File: ice5lp-dip40.sch (KiCad schematic (older format))
At the start: 34 parts

Commit message: Place all components on schematic
Parts:
- added J1: Conn_02x04_Odd_Even, esynr3z_Connector:PinHeader_2x04_P2.54mm_Vertical, symbol Connector_Generic:Conn_02x04_Odd_Even
- added J2, J3: Conn_01x20, esynr3z_Connector:PinHeader_1x20_P2.54mm_Vertical, symbol Connector_Generic:Conn_01x20
- gave numbers to parts that had none: 34
Connections:
- net labels added: +3V3, FLASH_MISO, FLASH_MOSI, ICE_CSN, ICE_SCK, IOB_0A, IOB_13B, IOB_16A, IOB_18A, IOB_20A, IOB_22A, IOB_23B, IOB_24A, IOB_25B, IOB_29B, IOB_2A, IOB_31B, IOB_3B, IOB_4A, IOB_5B, IOB_6A, IOB_8A, IOB_9B, IOT_36B, IOT_37A, IOT_38B, IOT_39A, IOT_41A, IOT_42B, IOT_43A, IOT_44B, IOT_45A, IOT_46B, IOT_48B, IOT_49A, IOT_50B, IOT_51A
- net labels removed: SPI_CSN, SPI_MISO, SPI_MOSI, SPI_SCK
- wire segments 130 -> 172
Other:
- note added: "IO"
- note added: "Power"
- note added: "Programming"

Commit message: Add RGB LED and assign some FPGA IO to pin headers
Parts:
- removed D2: LED_ARGB, symbol Device:LED_ARGB
- added D?: CLMVC-FKC-CGJJM569aBB7a343, esynr3z_LED:LED_Cree-PLCC4_2x2mm_CW, symbol esynr3z_LED:CLMVC-FKC-CGJJM569aBB7a343
- R7: value 1k -> 82
- R8, R9: value 1k -> 22
Connections:
- net labels added: IOB_36B, IOB_37A, IOB_38B, IOB_39A, IOB_41A, IOB_42B, IOB_43A, IOB_44B, IOB_45A, IOB_46B, IOB_48B, IOB_50B
- wire segments 172 -> 195
Changed lines of the file:
@@
 	9000 1300 9000 1350
-$Comp
-L Device:LED_ARGB D2
-U 1 1 5B47C861
-P 9400 3250
-F 0 "D2" H 9400 3747 50  0000 C CNN
-F 1 "LED_ARGB" H 9400 3656 50  0000 C CNN
-F 2 "" H 9400 3200 50  0001 C CNN
-F 3 "~" H 9400 3200 50  0001 C CNN
-	1    9400 3250
-	-1   0    0    -1
-$EndComp
 $Comp
 L power:+3.3V #PWR0125
@@
 P 9800 3050
 F 0 "R7" V 9900 3150 50  0000 C CNN
-F 1 "1k" V 9900 3000 50  0000 C CNN
+F 1 "82" V 9900 3000 50  0000 C CNN
 F 2 "" V 9730 3050 50  0001 C CNN
 F 3 "~" H 9800 3050 50  0001 C CNN
@@
 P 9800 3250
 F 0 "R8" V 9700 3150 50  0000 C CNN
-F 1 "1k" V 9700 3300 50  0000 C CNN
+F 1 "22" V 9700 3300 50  0000 C CNN
 F 2 "" V 9730 3250 50  0001 C CNN
 F 3 "~" H 9800 3250 50  0001 C CNN
@@
 P 9800 3450
 F 0 "R9" V 9700 3350 50  0000 C CNN
-F 1 "1k" V 9700 3500 50  0000 C CNN
+F 1 "22" V 9700 3500 50  0000 C CNN
 F 2 "" V 9730 3450 50  0001 C CNN
 F 3 "~" H 9800 3450 50  0001 C CNN
@@
 	6150 7650 6150 6450
 Wire Notes Line width 20
-	6150 6450 3850 6450
-Wire Notes Line width 20
-	3850 6450 3850 4150
-Wire Notes Line width 20
-	3850 4150 600  4150
+	6150 6450 4250 6450
+Wire Notes Line width 20
+	4250 6450 4250 4150
+Wire Notes Line width 20
+	4250 4150 600  4150
 Wire Notes Line width 20
 	600  4150 600  7650
@@
 Text Notes 8450 950  0    197  ~ 0
 IO
+$Comp
+L power:GND #PWR?
+U 1 1 5B6F631A
+P 9850 6000
+F 0 "#PWR?" H 9850 5750 50  0001 C CNN
+F 1 "GND" H 9855 5827 50  0000 C CNN
+F 2 "" H 9850 6000 50  0001 C CNN
+F 3 "" H 9850 6000 50  0001 C CNN
+	1    9850 6000
+	1    0    0    -1
+$EndComp
+$Comp
+L power:+5V #PWR?
+U 1 1 5B70EB47
+P 9850 5900
+F 0 "#PWR?" H 9850 5750 50  0001 C CNN
+F 1 "+5V" H 9865 6073 50  0000 C CNN
+F 2 "" H 9850 5900 50  0001 C CNN
+F 3 "" H 9850 5900 50  0001 C CNN
+	1    9850 5900
+	1    0    0    -1
+$EndComp
+Wire Wire Line
+	9250 6000 9850 6000
+Wire Wire Line
+	9850 5900 9250 5900
+$Comp
+L power:GND #PWR?
+U 1 1 5B71EE8C
+P 10700 6000
+F 0 "#PWR?" H 10700 5750 50  0001 C CNN
+F 1 "GND" H 10705 5827 50  0000 C CNN
+F 2 "" H 10700 6000 50  0001 C CNN
+F 3 "" H 10700 6000 50  0001 C CNN
+	1    10700 6000
+	1    0    0    -1
+$EndComp
+$Comp
+L power:+5V #PWR?
+U 1 1 5B71EE92
+P 10700 5900
+F 0 "#PWR?" H 10700 5750 50  0001 C CNN
+F 1 "+5V" H 10715 6073 50  0000 C CNN
+F 2 "" H 10700 5900 50  0001 C CNN
+F 3 "" H 10700 5900 50  0001 C CNN
+	1    10700 5900
+	1    0    0    -1
+$EndComp
+Wire Wire Line
+	10350 6000 10700 6000
+Wire Wire Line
+	10700 5900 10350 5900
+$Comp
+L power:GND #PWR?
+U 1 1 5B72752F
+P 9850 4100
+F 0 "#PWR?" H 9850 3850 50  0001 C CNN
+F 1 "GND" H 9855 3927 50  0000 C CNN
+F 2 "" H 9850 4100 50  0001 C CNN
+F 3 "" H 9850 4100 50  0001 C CNN
+	1    9850 4100
+	1    0    0    -1
+$EndComp
+Wire Wire Line
+	9250 4100 9850 4100
+$Comp
+L power:GND #PWR?
+U 1 1 5B72FA0D
+P 10700 4100
+F 0 "#PWR?" H 10700 3850 50  0001 C CNN
+F 1 "GND" H 10705 3927 50  0000 C CNN
+F 2 "" H 10700 4100 50  0001 C CNN
+F 3 "" H 10700 4100 50  0001 C CNN
+	1    10700 4100
+	1    0    0    -1
+$EndComp
+Wire Wire Line
+	10350 4100 10700 4100
+Text GLabel 9350 4200 2    50   Input ~ 0
+IOB_24A
+Wire Wire Line
+	9350 4200 9250 4200
+Text GLabel 9350 4300 2    50   Input ~ 0
+IOB_31B
+Wire Wire Line
+	9350 4300 9250 4300
+Text GLabel 9350 4400 2    50   Input ~ 0
+IOB_29B
+Wire Wire Line
+	9350 4400 9250 4400
+Text GLabel 9350 4500 2    50   Input ~ 0
+IOB_25B
+Wire Wire Line
+	9350 4500 9250 4500
+Text GLabel 9350 4600 2    50   Input ~ 0
+IOB_23B
+Wire Wire Line
+	9350 4600 9250 4600
+Text GLabel 9350 4700 2    50   Input ~ 0
+IOB_37A
+Wire Wire Line
+	9350 4700 9250 4700
+Text GLabel 9350 4800 2    50   Input ~ 0
+IOB_36B
+Wire Wire Line
+	9350 4800 9250 4800
+Text GLabel 9350 4900 2    50   Input ~ 0
+IOB_39A
+Wire Wire Line
+	9350 4900 9250 4900
+Text GLabel 9350 5000 2    50   Input ~ 0
+IOB_38B
+Wire Wire Line
+	9350 5000 9250 5000
+Text GLabel 9350 5100 2    50   Input ~ 0
+IOB_41A
+Wire Wire Line
+	9350 5100 9250 5100
+Text GLabel 9350 5200 2    50   Input ~ 0
+IOB_42B
+Wire Wire Line
+	9350 5200 9250 5200
+Text GLabel 9350 5300 2    50   Input ~ 0
+IOB_43A
+Wire Wire Line
+	9350 5300 9250 5300
+Text GLabel 9350 5400 2    50   Input ~ 0
+IOB_44B
+Wire Wire Line
+	9350 5400 9250 5400
+Text GLabel 9350 5500 2    50   Input ~ 0
+IOB_46B
+Wire Wire Line
+	9350 5500 9250 5500
+Text GLabel 9350 5600 2    50   Input ~ 0
+IOB_48B
+Wire Wire Line
+	9350 5600 9250 5600
+Text GLabel 9350 5700 2    50   Input ~ 0
+IOB_45A
+Wire Wire Line
+	9350 5700 9250 5700
+Text GLabel 9350 5800 2    50   Input ~ 0
+IOB_50B
+Wire Wire Line
+	9350 5800 9250 5800
+$Comp
+L esynr3z_LED:CLMVC-FKC-CGJJM569aBB7a343 D?
+U 1 1 5B843243
+P 9400 3250
+F 0 "D?" H 9400 3747 50  0000 C CNN
+F 1 "CLMVC-FKC-CGJJM569aBB7a343" H 9400 3656 50  0000 C CNN
+F 2 "esynr3z_LED:LED_Cree-PLCC4_2x2mm_CW" H 10200 3750 50  0001 C CNN
+F 3 "~" H 9400 3200 50  0001 C CNN
+	1    9400 3250
+	-1   0    0    -1
+$EndComp
 $EndSCHEMATC

Commit message: Add oscillator
Parts:
- removed D1: DIODE, symbol pspice:DIODE
- added C18, C19: 100n, symbol Device:C
- added D1: CDBU0520, esynr3z_Diode:SOD-523F, symbol esynr3z_DiodeRectifier:CDBU0520
- added D4: LED_RED, symbol Device:LED_ALT
- added D5: LED_ORANGE, symbol Device:LED_ALT
- added R11: 2.2k, symbol Device:R
- added R12: 10k, symbol Device:R
- added R13: 1k, symbol Device:R
- added SW2: SW_Push, symbol Switch:SW_Push
- added X1: ECS-2520MV-500-BN-TR, esynr3z_Oscillator:ECS-2520MV_4Pin_2.5x2.0mm, symbol esynr3z_Oscillator:ECS-2520MV-500-BN-TR
- D3: value LED_ALT -> LED_GREEN
- gave numbers to parts that had none: 1
Connections:
- net labels added: ICE_BTN, ICE_CLK, ICE_LED
- net labels removed: IOB_25B, IOB_36B, IOB_37A, IOB_38B, IOB_39A, IOB_41A, IOB_43A, IOB_44B, IOB_45A, IOB_46B, IOB_48B, IOB_50B
- wire segments 195 -> 218

Commit message: Add USB connector
Parts:
- added C?: 10u, symbol Device:C
- added J?: USB_B_Micro, esynr3z_ConnectorUSB:USB_Micro-B_Wurth_629105136821, symbol Connector:USB_B_Micro
Connections:
- wire segments 218 -> 226

Commit message: Add footprints to some symbols and trace pin headers and buttons
Parts:
- C17, C19, D3, R10, R12, R6, R7, R8, R9: footprint (none) -> esynr3z_Passive:0603
- SW1, SW2: footprint (none) -> esynr3z_Switch:PTS830
- gave numbers to parts that had none: 2
Connections:
- net labels added: RGB_B, RGB_G, RGB_R
- net labels removed: IOB_42B, IOT_50B, RGB0, RGB1, RGB2
- wire segments 226 -> 244
Changed lines of the file:
@@
 Text GLabel 6450 1350 1    50   Input ~ 0
 VCC_CORE
-Text GLabel 6250 1350 1    50   Input ~ 0
-VCC_PLL
-Wire Wire Line
-	6250 1450 6250 1350
 Wire Wire Line
 	6050 1400 6050 1450
@@
 F 0 "D3" V 3488 5682 50  0000 R CNN
 F 1 "LED_GREEN" V 3397 5682 50  0000 R CNN
-F 2 "" H 3450 5800 50  0001 C CNN
+F 2 "esynr3z_Passive:0603" H 3450 5800 50  0001 C CNN
 F 3 "~" H 3450 5800 50  0001 C CNN
 	1    3450 5800
@@
 F 0 "R10" H 3520 5446 50  0000 L CNN
 F 1 "1k" H 3520 5355 50  0000 L CNN
-F 2 "" V 3380 5400 50  0001 C CNN
+F 2 "esynr3z_Passive:0603" V 3380 5400 50  0001 C CNN
 F 3 "~" H 3450 5400 50  0001 C CNN
 	1    3450 5400
@@
 F 0 "SW1" V 3550 4250 50  0000 R CNN
 F 1 "SW_Push" V 3450 4450 50  0000 R CNN
-F 2 "" H 3500 4200 50  0001 C CNN
+F 2 "esynr3z_Switch:PTS830" H 3500 4200 50  0001 C CNN
 F 3 "" H 3500 4200 50  0001 C CNN
 	1    3500 4000
@@
 F 0 "R6" H 3570 3596 50  0000 L CNN
 F 1 "10k" H 3570 3505 50  0000 L CNN
-F 2 "" V 3430 3550 50  0001 C CNN
+F 2 "esynr3z_Passive:0603" V 3430 3550 50  0001 C CNN
 F 3 "~" H 3500 3550 50  0001 C CNN
 	1    3500 3550
@@
 F 0 "C17" H 3915 3996 50  0000 L CNN
 F 1 "100n" H 3915 3905 50  0000 L CNN
-F 2 "" H 3838 3800 50  0001 C CNN
+F 2 "esynr3z_Passive:0603" H 3838 3800 50  0001 C CNN
 F 3 "~" H 3800 3950 50  0001 C CNN
 	1    3800 3950
@@
 	9300 3100 9400 3100
 Text GLabel 7600 4850 2    50   Input ~ 0
-RGB0
+RGB_R
 Text GLabel 7600 4950 2    50   Input ~ 0
-RGB1
+RGB_G
 Text GLabel 7600 5050 2    50   Input ~ 0
-RGB2
+RGB_B
 Wire Wire Line
 	7600 5050 7500 5050
@@
 F 0 "R7" V 10100 3000 50  0000 C CNN
 F 1 "82" V 10100 2850 50  0000 C CNN
-F 2 "" V 9930 2900 50  0001 C CNN
+F 2 "esynr3z_Passive:0603" V 9930 2900 50  0001 C CNN
 F 3 "~" H 10000 2900 50  0001 C CNN
 	1    10000 2900
@@
 F 0 "R8" V 9900 3000 50  0000 C CNN
 F 1 "22" V 9900 3150 50  0000 C CNN
-F 2 "" V 9930 3100 50  0001 C CNN
+F 2 "esynr3z_Passive:0603" V 9930 3100 50  0001 C CNN
 F 3 "~" H 10000 3100 50  0001 C CNN
 	1    10000 3100
@@
 F 0 "R9" V 9900 3200 50  0000 C CNN
 F 1 "22" V 9900 3350 50  0000 C CNN
-F 2 "" V 9930 3300 50  0001 C CNN
+F 2 "esynr3z_Passive:0603" V 9930 3300 50  0001 C CNN
 F 3 "~" H 10000 3300 50  0001 C CNN
 	1    10000 3300
@@
 	9800 3300 9850 3300
 Text GLabel 10200 2900 2    50   Input ~ 0
-RGB0
+RGB_R
 Text GLabel 10200 3100 2    50   Input ~ 0
-RGB1
+RGB_G
 Text GLabel 10200 3300 2    50   Input ~ 0
-RGB2
+RGB_B
 Wire Wire Line
 	10200 2900 10150 2900
@@
 IOT_49A
 Text GLabel 7600 4550 2    50   Input ~ 0
-IOT_50B
+ICE_BTN
 Text GLabel 7600 4650 2    50   Input ~ 0
 IOT_51A
@@
 L power:GND #PWR0140
 U 1 1 5B71EE8C
-P 10700 6000
-F 0 "#PWR0140" H 10700 5750 50  0001 C CNN
-F 1 "GND" H 10705 5827 50  0000 C CNN
-F 2 "" H 10700 6000 50  0001 C CNN
-F 3 "" H 10700 6000 50  0001 C CNN
-	1    10700 6000
+P 10950 6000
+F 0 "#PWR0140" H 10950 5750 50  0001 C CNN
+F 1 "GND" H 10955 5827 50  0000 C CNN
+F 2 "" H 10950 6000 50  0001 C CNN
+F 3 "" H 10950 6000 50  0001 C CNN
+	1    10950 6000
 	1    0    0    -1
 $EndComp
@@
 L power:+5V #PWR0141
 U 1 1 5B71EE92
-P 10700 5900
-F 0 "#PWR0141" H 10700 5750 50  0001 C CNN
-F 1 "+5V" H 10715 6073 50  0000 C CNN
-F 2 "" H 10700 5900 50  0001 C CNN
-F 3 "" H 10700 5900 50  0001 C CNN
-	1    10700 5900
-	1    0    0    -1
-$EndComp
-Wire Wire Line
-	10350 6000 10700 6000
-Wire Wire Line
-	10700 5900 10350 5900
+P 10950 5900
+F 0 "#PWR0141" H 10950 5750 50  0001 C CNN
+F 1 "+5V" H 10965 6073 50  0000 C CNN
+F 2 "" H 10950 5900 50  0001 C CNN
+F 3 "" H 10950 5900 50  0001 C CNN
+	1    10950 5900
+	1    0    0    -1
+$EndComp
+Wire Wire Line
+	10350 6000 10950 6000
+Wire Wire Line
+	10950 5900 10350 5900
 $Comp
 L power:GND #PWR0142
@@
 L power:GND #PWR0143
 U 1 1 5B72FA0D
-P 10700 4100
-F 0 "#PWR0143" H 10700 3850 50  0001 C CNN
-F 1 "GND" H 10705 3927 50  0000 C CNN
-F 2 "" H 10700 4100 50  0001 C CNN
-F 3 "" H 10700 4100 50  0001 C CNN
-	1    10700 4100
-	1    0    0    -1
-$EndComp
-Wire Wire Line
-	10350 4100 10700 4100
-Text GLabel 9350 4200 2    50   Input ~ 0
+P 10950 4100
+F 0 "#PWR0143" H 10950 3850 50  0001 C CNN
+F 1 "GND" H 10955 3927 50  0000 C CNN
+F 2 "" H 10950 4100 50  0001 C CNN
+F 3 "" H 10950 4100 50  0001 C CNN
+	1    10950 4100
+	1    0    0    -1
+$EndComp
+Wire Wire Line
+	10350 4100 10950 4100
+Text GLabel 9350 4300 2    50   Input ~ 0
 IOB_24A
 Wire Wire Line
 	9350 4200 9250 4200
-Text GLabel 9350 4300 2    50   Input ~ 0
+Text GLabel 9350 4400 2    50   Input ~ 0
 IOB_31B
 Wire Wire Line
 	9350 4300 9250 4300
-Text GLabel 9350 4400 2    50   Input ~ 0
+Text GLabel 9350 4500 2    50   Input ~ 0
 IOB_29B
 Wire Wire Line
@@
 	9350 5100 9250 5100
 Text GLabel 9350 5200 2    50   Input ~ 0
-IOB_42B
+IOT_42B
 Wire Wire Line
 	9350 5200 9250 5200
@@
 	9350 5700 9250 5700
 Text GLabel 9350 5800 2    50   Input ~ 0
-IOT_50B
+ICE_BTN
 Wire Wire Line
 	9350 5800 9250 5800
@@
 F 0 "SW2" V 8850 2150 50  0000 R CNN
 F 1 "SW_Push" V 8750 2350 50  0000 R CNN
-F 2 "" H 8800 2100 50  0001 C CNN
+F 2 "esynr3z_Switch:PTS830" H 8800 2100 50  0001 C CNN
 F 3 "" H 8800 2100 50  0001 C CNN
 	1    8800 1900
@@
 F 0 "R12" H 8870 1496 50  0000 L CNN
 F 1 "10k" H 8870 1405 50  0000 L CNN
-F 2 "" V 8730 1450 50  0001 C CNN
+F 2 "esynr3z_Passive:0603" V 8730 1450 50  0001 C CNN
 F 3 "~" H 8800 1450 50  0001 C CNN
 	1    8800 1450
@@
 F 0 "C19" H 9215 1896 50  0000 L CNN
 F 1 "100n" H 9215 1805 50  0000 L CNN
-F 2 "" H 9138 1700 50  0001 C CNN
+F 2 "esynr3z_Passive:0603" H 9138 1700 50  0001 C CNN
 F 3 "~" H 9100 1850 50  0001 C CNN
 	1    9100 1850
@@
 	10300 1400 10300 1450
 $Comp
-L power:GND #PWR?
+L power:GND #PWR0151
 U 1 1 5BB52FA7
 P 1350 4100
-F 0 "#PWR?" H 1350 3850 50  0001 C CNN
+F 0 "#PWR0151" H 1350 3850 50  0001 C CNN
 F 1 "GND" H 1355 3927 50  0000 C CNN
 F 2 "" H 1350 4100 50  0001 C CNN
@@
 $EndComp
 $Comp
-L power:+5V #PWR?
+L power:+5V #PWR0153
 U 1 1 5BB7791B
 P 1900 3350
-F 0 "#PWR?" H 1900 3200 50  0001 C CNN
+F 0 "#PWR0153" H 1900 3200 50  0001 C CNN
 F 1 "+5V" H 1915 3523 50  0000 C CNN
 F 2 "" H 1900 3350 50  0001 C CNN
@@
 	1900 3400 1900 3350
 $Comp
-L Device:C C?
+L Device:C C20
 U 1 1 5BB9F4F5
 P 1900 3750
-F 0 "C?" H 2015 3796 50  0000 L CNN
+F 0 "C20" H 2015 3796 50  0000 L CNN
 F 1 "10u" H 2015 3705 50  0000 L CNN
 F 2 "" H 1938 3600 50  0001 C CNN
@@
 $EndComp
 $Comp
-L power:GND #PWR?
+L power:GND #PWR0154
 U 1 1 5BB9F4FC
 P 1900 4100
-F 0 "#PWR?" H 1900 3850 50  0001 C CNN
+F 0 "#PWR0154" H 1900 3850 50  0001 C CNN
 F 1 "GND" H 1905 3927 50  0000 C CNN
 F 2 "" H 1900 4100 50  0001 C CNN
@@
 	2600 3400 2600 3650
 $Comp
-L Connector:USB_B_Micro J?
+L Connector:USB_B_Micro J4
 U 1 1 5BB09EED
 P 1350 3600
-F 0 "J?" H 1405 4067 50  0000 C CNN
+F 0 "J4" H 1405 4067 50  0000 C CNN
 F 1 "USB_B_Micro" H 1405 3976 50  0000 C CNN
 F 2 "esynr3z_ConnectorUSB:USB_Micro-B_Wurth_629105136821" H 1500 3550 50  0001 C CNN
@@
 Wire Wire Line
 	1350 4050 1350 4100
+Text GLabel 9350 4200 2    50   Input ~ 0
+IOB_22A
+Text GLabel 10450 4200 2    50   Input ~ 0
+IOB_20A
+Wire Wire Line
+	10450 4200 10350 4200
+Text GLabel 10450 4300 2    50   Input ~ 0
+IOB_18A
+Wire Wire Line
+	10450 4300 10350 4300
+Text GLabel 10450 4400 2    50   Input ~ 0
+IOB_16A
+Wire Wire Line
+	10450 4400 10350 4400
+Text GLabel 10450 4500 2    50   Input ~ 0
+IOB_13B
+Wire Wire Line
+	10450 4500 10350 4500
+Text GLabel 10450 4600 2    50   Input ~ 0
+IOB_8A
+Wire Wire Line
+	10450 4600 10350 4600
+Text GLabel 10450 4700 2    50   Input ~ 0
+IOB_9B
+Wire Wire Line
+	10450 4700 10350 4700
+Text GLabel 10450 4800 2    50   Input ~ 0
+IOB_6A
+Wire Wire Line
+	10450 4800 10350 4800
+Text GLabel 10450 4900 2    50   Input ~ 0
+IOB_4A
+Wire Wire Line
+	10450 4900 10350 4900
+Text GLabel 10450 5000 2    50   Input ~ 0
+IOB_2A
+Wire Wire Line
+	10450 5000 10350 5000
+Text GLabel 10450 5100 2    50   Input ~ 0
+IOB_0A
+Wire Wire Line
+	10450 5100 10350 5100
+Text GLabel 10450 5200 2    50   Input ~ 0
+IOB_5B
+Wire Wire Line
+	10450 5200 10350 5200
+Text GLabel 10450 5300 2    50   Input ~ 0
+IOB_3B
+Wire Wire Line
+	10450 5300 10350 5300
+Text GLabel 10450 5600 2    50   Input ~ 0
+RGB_R
+Wire Wire Line
+	10450 5400 10350 5400
+Text GLabel 10450 5700 2    50   Input ~ 0
+RGB_G
+Wire Wire Line
+	10450 5500 10350 5500
+Text GLabel 10450 5800 2    50   Input ~ 0
+RGB_B
+Wire Wire Line
+	10450 5600 10350 5600
+Text GLabel 10450 5400 2    50   Input ~ 0
+IOT_49A
+Wire Wire Line
+	10450 5700 10350 5700
+Text GLabel 10450 5500 2    50   Input ~ 0
+IOT_51A
+Wire Wire Line
+	10450 5800 10350 5800
+Wire Wire Line
+	6350 1400 6250 1400
+Connection ~ 6350 1400
+Wire Wire Line
+	6250 1400 6250 1450
 $EndSCHEMATC
