File: ice5lp-dip40.sch (KiCad schematic (older format))
At the start: 48 parts, among them J1 Conn_02x04_Odd_Even, J2 Conn_01x20, J3 Conn_01x20, J4 USB_B_Micro, SW1 SW_Push, SW2 SW_Push, U1 AT25D011-SSHF, U2 MIC5355-S4YMME, U3 ICE5LP4K-SG48, X1 ECS-2520MV-500-BN-TR

Commit message: Update footprints
Parts:
- C1, C10, C11, C12, C13, C14, C15, C16, C18, C2, C20, C3, C4, C5, C6, C7, C8, C9: footprint (none) -> esynr3z_Capacitor:C_0603
- C17, C19: footprint esynr3z_Passive:0603 -> esynr3z_Capacitor:C_0603
- D3: footprint esynr3z_Passive:0603 -> esynr3z_LED:LED_0603
- D4, D5: footprint (none) -> esynr3z_LED:LED_0603
- R1, R11, R13, R2, R3, R4, R5: footprint (none) -> esynr3z_Resistor:R_0603
- R10, R12, R6, R7, R8, R9: footprint esynr3z_Passive:0603 -> esynr3z_Resistor:R_0603
Changed lines of the file:
@@
 F 0 "C5" H 2315 7196 50  0000 L CNN
 F 1 "1u" H 2315 7105 50  0000 L CNN
-F 2 "" H 2238 7000 50  0001 C CNN
+F 2 "esynr3z_Capacitor:C_0603" H 2238 7000 50  0001 C CNN
 F 3 "~" H 2200 7150 50  0001 C CNN
 	1    2200 7150
@@
 F 0 "C6" H 2665 7196 50  0000 L CNN
 F 1 "100n" H 2665 7105 50  0000 L CNN
-F 2 "" H 2588 7000 50  0001 C CNN
+F 2 "esynr3z_Capacitor:C_0603" H 2588 7000 50  0001 C CNN
 F 3 "~" H 2550 7150 50  0001 C CNN
 	1    2550 7150
@@
 F 0 "R3" H 2130 6704 50  0000 R CNN
 F 1 "100" H 2130 6795 50  0000 R CNN
-F 2 "" V 2130 6750 50  0001 C CNN
+F 2 "esynr3z_Resistor:R_0603" V 2130 6750 50  0001 C CNN
 F 3 "~" H 2200 6750 50  0001 C CNN
 	1    2200 6750
@@
 F 0 "C1" H 865 7196 50  0000 L CNN
 F 1 "1u" H 865 7105 50  0000 L CNN
-F 2 "" H 788 7000 50  0001 C CNN
+F 2 "esynr3z_Capacitor:C_0603" H 788 7000 50  0001 C CNN
 F 3 "~" H 750 7150 50  0001 C CNN
 	1    750  7150
@@
 F 0 "C2" H 1215 7196 50  0000 L CNN
 F 1 "100n" H 1215 7105 50  0000 L CNN
-F 2 "" H 1138 7000 50  0001 C CNN
+F 2 "esynr3z_Capacitor:C_0603" H 1138 7000 50  0001 C CNN
 F 3 "~" H 1100 7150 50  0001 C CNN
 	1    1100 7150
@@
 F 0 "C4" H 1615 7196 50  0000 L CNN
 F 1 "100n" H 1615 7105 50  0000 L CNN
-F 2 "" H 1538 7000 50  0001 C CNN
+F 2 "esynr3z_Capacitor:C_0603" H 1538 7000 50  0001 C CNN
 F 3 "~" H 1500 7150 50  0001 C CNN
 	1    1500 7150
@@
 F 0 "C15" H 5300 1250 50  0000 L CNN
 F 1 "100n" H 5250 1150 50  0000 L CNN
-F 2 "" H 5588 1050 50  0001 C CNN
+F 2 "esynr3z_Capacitor:C_0603" H 5588 1050 50  0001 C CNN
 F 3 "~" H 5550 1200 50  0001 C CNN
 	1    5550 1200
@@
 F 0 "C9" H 3315 7196 50  0000 L CNN
 F 1 "1u" H 3315 7105 50  0000 L CNN
-F 2 "" H 3238 7000 50  0001 C CNN
+F 2 "esynr3z_Capacitor:C_0603" H 3238 7000 50  0001 C CNN
 F 3 "~" H 3200 7150 50  0001 C CNN
 	1    3200 7150
@@
 F 0 "C11" H 3665 7196 50  0000 L CNN
 F 1 "100n" H 3665 7105 50  0000 L CNN
-F 2 "" H 3588 7000 50  0001 C CNN
+F 2 "esynr3z_Capacitor:C_0603" H 3588 7000 50  0001 C CNN
 F 3 "~" H 3550 7150 50  0001 C CNN
 	1    3550 7150
@@
 F 0 "C12" H 4315 7196 50  0000 L CNN
 F 1 "1u" H 4315 7105 50  0000 L CNN
-F 2 "" H 4238 7000 50  0001 C CNN
+F 2 "esynr3z_Capacitor:C_0603" H 4238 7000 50  0001 C CNN
 F 3 "~" H 4200 7150 50  0001 C CNN
 	1    4200 7150
@@
 F 0 "C13" H 4665 7196 50  0000 L CNN
 F 1 "100n" H 4665 7105 50  0000 L CNN
-F 2 "" H 4588 7000 50  0001 C CNN
+F 2 "esynr3z_Capacitor:C_0603" H 4588 7000 50  0001 C CNN
 F 3 "~" H 4550 7150 50  0001 C CNN
 	1    4550 7150
@@
 F 0 "C14" H 5315 7196 50  0000 L CNN
 F 1 "1u" H 5315 7105 50  0000 L CNN
-F 2 "" H 5238 7000 50  0001 C CNN
+F 2 "esynr3z_Capacitor:C_0603" H 5238 7000 50  0001 C CNN
 F 3 "~" H 5200 7150 50  0001 C CNN
 	1    5200 7150
@@
 F 0 "C16" H 5665 7196 50  0000 L CNN
 F 1 "100n" H 5665 7105 50  0000 L CNN
-F 2 "" H 5588 7000 50  0001 C CNN
+F 2 "esynr3z_Capacitor:C_0603" H 5588 7000 50  0001 C CNN
 F 3 "~" H 5550 7150 50  0001 C CNN
 	1    5550 7150
@@
 F 0 "D3" V 3488 5682 50  0000 R CNN
 F 1 "LED_GREEN" V 3397 5682 50  0000 R CNN
-F 2 "esynr3z_Passive:0603" H 3450 5800 50  0001 C CNN
+F 2 "esynr3z_LED:LED_0603" H 3450 5800 50  0001 C CNN
 F 3 "~" H 3450 5800 50  0001 C CNN
 	1    3450 5800
@@
 F 0 "R10" H 3520 5446 50  0000 L CNN
 F 1 "1k" H 3520 5355 50  0000 L CNN
-F 2 "esynr3z_Passive:0603" V 3380 5400 50  0001 C CNN
+F 2 "esynr3z_Resistor:R_0603" V 3380 5400 50  0001 C CNN
 F 3 "~" H 3450 5400 50  0001 C CNN
 	1    3450 5400
@@
 F 0 "R6" H 3570 3596 50  0000 L CNN
 F 1 "10k" H 3570 3505 50  0000 L CNN
-F 2 "esynr3z_Passive:0603" V 3430 3550 50  0001 C CNN
+F 2 "esynr3z_Resistor:R_0603" V 3430 3550 50  0001 C CNN
 F 3 "~" H 3500 3550 50  0001 C CNN
 	1    3500 3550
@@
 F 0 "C17" H 3915 3996 50  0000 L CNN
 F 1 "100n" H 3915 3905 50  0000 L CNN
-F 2 "esynr3z_Passive:0603" H 3838 3800 50  0001 C CNN
+F 2 "esynr3z_Capacitor:C_0603" H 3838 3800 50  0001 C CNN
 F 3 "~" H 3800 3950 50  0001 C CNN
 	1    3800 3950
@@
 F 0 "R7" V 10100 3000 50  0000 C CNN
 F 1 "82" V 10100 2850 50  0000 C CNN
-F 2 "esynr3z_Passive:0603" V 9930 2900 50  0001 C CNN
+F 2 "esynr3z_Resistor:R_0603" V 9930 2900 50  0001 C CNN
 F 3 "~" H 10000 2900 50  0001 C CNN
 	1    10000 2900
@@
 F 0 "R8" V 9900 3000 50  0000 C CNN
 F 1 "22" V 9900 3150 50  0000 C CNN
-F 2 "esynr3z_Passive:0603" V 9930 3100 50  0001 C CNN
+F 2 "esynr3z_Resistor:R_0603" V 9930 3100 50  0001 C CNN
 F 3 "~" H 10000 3100 50  0001 C CNN
 	1    10000 3100
@@
 F 0 "R9" V 9900 3200 50  0000 C CNN
 F 1 "22" V 9900 3350 50  0000 C CNN
-F 2 "esynr3z_Passive:0603" V 9930 3300 50  0001 C CNN
+F 2 "esynr3z_Resistor:R_0603" V 9930 3300 50  0001 C CNN
 F 3 "~" H 10000 3300 50  0001 C CNN
 	1    10000 3300
@@
 F 0 "C3" H 865 5796 50  0000 L CNN
 F 1 "2.2u" H 865 5705 50  0000 L CNN
-F 2 "" H 788 5600 50  0001 C CNN
+F 2 "esynr3z_Capacitor:C_0603" H 788 5600 50  0001 C CNN
 F 3 "~" H 750 5750 50  0001 C CNN
 	1    750  5750
@@
 F 0 "C7" H 2315 5796 50  0000 L CNN
 F 1 "2.2u" H 2315 5705 50  0000 L CNN
-F 2 "" H 2238 5600 50  0001 C CNN
+F 2 "esynr3z_Capacitor:C_0603" H 2238 5600 50  0001 C CNN
 F 3 "~" H 2200 5750 50  0001 C CNN
 	1    2200 5750
@@
 F 0 "C8" H 2715 5796 50  0000 L CNN
 F 1 "2.2u" H 2715 5705 50  0000 L CNN
-F 2 "" H 2638 5600 50  0001 C CNN
+F 2 "esynr3z_Capacitor:C_0603" H 2638 5600 50  0001 C CNN
 F 3 "~" H 2600 5750 50  0001 C CNN
 	1    2600 5750
@@
 F 0 "C10" H 3400 1450 50  0000 L CNN
 F 1 "100n" H 3400 1350 50  0000 L CNN
-F 2 "" H 3288 1250 50  0001 C CNN
+F 2 "esynr3z_Capacitor:C_0603" H 3288 1250 50  0001 C CNN
 F 3 "~" H 3250 1400 50  0001 C CNN
 	1    3250 1400
@@
 F 0 "R2" H 1520 1446 50  0000 L CNN
 F 1 "10k" H 1520 1355 50  0000 L CNN
-F 2 "" V 1380 1400 50  0001 C CNN
+F 2 "esynr3z_Resistor:R_0603" V 1380 1400 50  0001 C CNN
 F 3 "~" H 1450 1400 50  0001 C CNN
 	1    1450 1400
@@
 F 0 "R4" H 2670 1446 50  0000 L CNN
 F 1 "10k" H 2670 1355 50  0000 L CNN
-F 2 "" V 2530 1400 50  0001 C CNN
+F 2 "esynr3z_Resistor:R_0603" V 2530 1400 50  0001 C CNN
 F 3 "~" H 2600 1400 50  0001 C CNN
 	1    2600 1400
@@
 F 0 "R5" H 2970 1446 50  0000 L CNN
 F 1 "10k" H 2970 1355 50  0000 L CNN
-F 2 "" V 2830 1400 50  0001 C CNN
+F 2 "esynr3z_Resistor:R_0603" V 2830 1400 50  0001 C CNN
 F 3 "~" H 2900 1400 50  0001 C CNN
 	1    2900 1400
@@
 F 0 "R1" H 1220 1446 50  0000 L CNN
 F 1 "10k" H 1220 1355 50  0000 L CNN
-F 2 "" V 1080 1400 50  0001 C CNN
+F 2 "esynr3z_Resistor:R_0603" V 1080 1400 50  0001 C CNN
 F 3 "~" H 1150 1400 50  0001 C CNN
 	1    1150 1400
@@
 F 0 "C18" H 4150 6000 50  0000 L CNN
 F 1 "100n" H 4100 5900 50  0000 L CNN
-F 2 "" H 4438 5800 50  0001 C CNN
+F 2 "esynr3z_Capacitor:C_0603" H 4438 5800 50  0001 C CNN
 F 3 "~" H 4400 5950 50  0001 C CNN
 	1    4400 5950
@@
 F 0 "R12" H 8870 1496 50  0000 L CNN
 F 1 "10k" H 8870 1405 50  0000 L CNN
-F 2 "esynr3z_Passive:0603" V 8730 1450 50  0001 C CNN
+F 2 "esynr3z_Resistor:R_0603" V 8730 1450 50  0001 C CNN
 F 3 "~" H 8800 1450 50  0001 C CNN
 	1    8800 1450
@@
 F 0 "C19" H 9215 1896 50  0000 L CNN
 F 1 "100n" H 9215 1805 50  0000 L CNN
-F 2 "esynr3z_Passive:0603" H 9138 1700 50  0001 C CNN
+F 2 "esynr3z_Capacitor:C_0603" H 9138 1700 50  0001 C CNN
 F 3 "~" H 9100 1850 50  0001 C CNN
 	1    9100 1850
@@
 F 0 "D4" V 2638 3682 50  0000 R CNN
 F 1 "LED_RED" V 2547 3682 50  0000 R CNN
-F 2 "" H 2600 3800 50  0001 C CNN
+F 2 "esynr3z_LED:LED_0603" H 2600 3800 50  0001 C CNN
 F 3 "~" H 2600 3800 50  0001 C CNN
 	1    2600 3800
@@
 F 0 "R11" V 2150 3250 50  0000 L CNN
 F 1 "2.2k" V 2150 3450 50  0000 L CNN
-F 2 "" V 2180 3400 50  0001 C CNN
+F 2 "esynr3z_Resistor:R_0603" V 2180 3400 50  0001 C CNN
 F 3 "~" H 2250 3400 50  0001 C CNN
 	1    2250 3400
@@
 F 0 "D5" V 10338 1832 50  0000 R CNN
 F 1 "LED_ORANGE" V 10247 1832 50  0000 R CNN
-F 2 "" H 10300 1950 50  0001 C CNN
+F 2 "esynr3z_LED:LED_0603" H 10300 1950 50  0001 C CNN
 F 3 "~" H 10300 1950 50  0001 C CNN
 	1    10300 1950
@@
 F 0 "R13" H 10350 1650 50  0000 L CNN
 F 1 "1k" H 10350 1550 50  0000 L CNN
-F 2 "" V 10230 1600 50  0001 C CNN
+F 2 "esynr3z_Resistor:R_0603" V 10230 1600 50  0001 C CNN
 F 3 "~" H 10300 1600 50  0001 C CNN
 	1    10300 1600
@@
 F 0 "C20" H 2015 3796 50  0000 L CNN
 F 1 "10u" H 2015 3705 50  0000 L CNN
-F 2 "" H 1938 3600 50  0001 C CNN
+F 2 "esynr3z_Capacitor:C_0603" H 1938 3600 50  0001 C CNN
 F 3 "~" H 1900 3750 50  0001 C CNN
 	1    1900 3750

Commit message: Place and trace all main components
Connections:
- net labels removed: IOB_20A
Changed lines of the file:
@@
 Wire Wire Line
 	1850 2500 1900 2500
+Text GLabel 1800 2600 0    50   Input ~ 0
+CRESET
 Text GLabel 2500 2600 2    50   Input ~ 0
-CRESET
-Text GLabel 1800 2600 0    50   Input ~ 0
 CDONE
 Wire Wire Line
@@
 Wire Wire Line
 	1900 2600 1800 2600
+Text GLabel 2500 2700 2    50   Input ~ 0
+FLASH_MISO
+Text GLabel 1800 2800 0    50   Input ~ 0
+ICE_SCK
+Wire Wire Line
+	2500 2700 2400 2700
+Wire Wire Line
+	1800 2700 1900 2700
 Text GLabel 1800 2700 0    50   Input ~ 0
-FLASH_MISO
-Text GLabel 2500 2700 2    50   Input ~ 0
-ICE_SCK
-Wire Wire Line
-	2500 2700 2400 2700
-Wire Wire Line
-	1800 2700 1900 2700
-Text GLabel 1800 2800 0    50   Input ~ 0
 ICE_CSN
 Wire Wire Line
@@
 IOB_18A
 Text GLabel 4900 3700 0    50   Input ~ 0
-IOB_20A
+ICE_LED
 Text GLabel 4900 3800 0    50   Input ~ 0
 IOB_22A
@@
 IOB_22A
 Text GLabel 10450 4200 2    50   Input ~ 0
-IOB_20A
+ICE_LED
 Wire Wire Line
 	10450 4200 10350 4200

Commit message: Place some caps
Parts:
- removed C5: 1u, esynr3z_Capacitor:C_0603, symbol Device:C
- removed C6: 100n, esynr3z_Capacitor:C_0603, symbol Device:C
- removed R3: 100, esynr3z_Resistor:R_0603, symbol Device:R
Connections:
- net labels removed: VCC_PLL
- wire segments 244 -> 236
Changed lines of the file:
@@
 	1    0    0    -1
 $EndComp
-$Comp
-L power:+1V2 #PWR0102
-U 1 1 5B44F591
-P 2200 6550
-F 0 "#PWR0102" H 2200 6400 50  0001 C CNN
-F 1 "+1V2" H 2215 6723 50  0000 C CNN
-F 2 "" H 2200 6550 50  0001 C CNN
-F 3 "" H 2200 6550 50  0001 C CNN
-	1    2200 6550
-	1    0    0    -1
-$EndComp
-$Comp
-L Device:C C5
-U 1 1 5B44FA21
-P 2200 7150
-F 0 "C5" H 2315 7196 50  0000 L CNN
-F 1 "1u" H 2315 7105 50  0000 L CNN
-F 2 "esynr3z_Capacitor:C_0603" H 2238 7000 50  0001 C CNN
-F 3 "~" H 2200 7150 50  0001 C CNN
-	1    2200 7150
-	1    0    0    -1
-$EndComp
-$Comp
-L Device:C C6
-U 1 1 5B44FB29
-P 2550 7150
-F 0 "C6" H 2665 7196 50  0000 L CNN
-F 1 "100n" H 2665 7105 50  0000 L CNN
-F 2 "esynr3z_Capacitor:C_0603" H 2588 7000 50  0001 C CNN
-F 3 "~" H 2550 7150 50  0001 C CNN
-	1    2550 7150
-	1    0    0    -1
-$EndComp
-$Comp
-L Device:R R3
-U 1 1 5B44FB8D
-P 2200 6750
-F 0 "R3" H 2130 6704 50  0000 R CNN
-F 1 "100" H 2130 6795 50  0000 R CNN
-F 2 "esynr3z_Resistor:R_0603" V 2130 6750 50  0001 C CNN
-F 3 "~" H 2200 6750 50  0001 C CNN
-	1    2200 6750
-	-1   0    0    1
-$EndComp
-$Comp
-L power:GND #PWR0103
-U 1 1 5B4503A1
-P 2200 7350
-F 0 "#PWR0103" H 2200 7100 50  0001 C CNN
-F 1 "GND" H 2205 7177 50  0000 C CNN
-F 2 "" H 2200 7350 50  0001 C CNN
-F 3 "" H 2200 7350 50  0001 C CNN
-	1    2200 7350
-	1    0    0    -1
-$EndComp
-$Comp
-L power:GND #PWR0104
-U 1 1 5B450405
-P 2550 7350
-F 0 "#PWR0104" H 2550 7100 50  0001 C CNN
-F 1 "GND" H 2555 7177 50  0000 C CNN
-F 2 "" H 2550 7350 50  0001 C CNN
-F 3 "" H 2550 7350 50  0001 C CNN
-	1    2550 7350
-	1    0    0    -1
-$EndComp
-Wire Wire Line
-	2550 7350 2550 7300
-Wire Wire Line
-	2200 7350 2200 7300
-Wire Wire Line
-	2200 6550 2200 6600
-Wire Wire Line
-	2200 6950 2550 6950
-Wire Wire Line
-	2550 6950 2550 7000
 Wire Wire Line
 	6450 1350 6450 1400
@@
 Wire Wire Line
 	6050 800  6050 900
-Wire Wire Line
-	2200 6900 2200 6950
-Connection ~ 2200 6950
-Wire Wire Line
-	2200 6950 2200 7000
-Text GLabel 2650 6950 2    50   Input ~ 0
-VCC_PLL
-Wire Wire Line
-	2650 6950 2550 6950
-Connection ~ 2550 6950
 $Comp
 L power:+1V2 #PWR0106
