File: ice40-dip40.sch (KiCad schematic (older format))
At the start: 46 parts, among them J1 Conn_02x04_Odd_Even, J2 Conn_01x20, J3 Conn_01x20, J4 USB_B_Micro, SW1 SW_Push, SW2 SW_Push, U1 AT25D081-SSHD, U2 MIC5355-S4YMME, U3 ICE5LP4K-SG48, X1 ECS-2520MV-120-BN-TR

Commit message: Project rename
Parts:
- C1, C10, C11, C12, C13, C15, C17, C18, C19, C2, C20, C3, C4, C7, C8, C9: symbol ice5lp-dip40:Device_C -> ice40-dip40:Device_C
- D1: symbol ice5lp-dip40:esynr3z_DiodeRectifier_CDBU0520 -> ice40-dip40:esynr3z_DiodeRectifier_CDBU0520
- D2: symbol ice5lp-dip40:esynr3z_LED_CLMVC-FKC-CGJJM569aBB7a343 -> ice40-dip40:esynr3z_LED_CLMVC-FKC-CGJJM569aBB7a343
- D3, D4, D5: symbol ice5lp-dip40:Device_LED_ALT -> ice40-dip40:Device_LED_ALT
- J1: symbol ice5lp-dip40:Connector_Generic_Conn_02x04_Odd_Even -> ice40-dip40:Connector_Generic_Conn_02x04_Odd_Even
- J2, J3: symbol ice5lp-dip40:Connector_Generic_Conn_01x20 -> ice40-dip40:Connector_Generic_Conn_01x20
- J4: symbol ice5lp-dip40:Connector_USB_B_Micro -> ice40-dip40:Connector_USB_B_Micro
- R1, R10, R11, R12, R13, R14, R15, R2, R3, R4, R5, R6, R7, R8, R9: symbol ice5lp-dip40:Device_R -> ice40-dip40:Device_R
- SW1, SW2: symbol ice5lp-dip40:Switch_SW_Push -> ice40-dip40:Switch_SW_Push
- U1: symbol ice5lp-dip40:esynr3z_MemoryFlash_AT25D081-SSHD -> ice40-dip40:esynr3z_MemoryFlash_AT25D081-SSHD
- U2: symbol ice5lp-dip40:esynr3z_RegulatorLinear_MIC5355-S4YMME -> ice40-dip40:esynr3z_RegulatorLinear_MIC5355-S4YMME
- U3: symbol ice5lp-dip40:esynr3z_FPGA_ICE5LP4K-SG48 -> ice40-dip40:esynr3z_FPGA_ICE5LP4K-SG48
- X1: symbol ice5lp-dip40:esynr3z_Oscillator_ECS-2520MV-XXX -> ice40-dip40:esynr3z_Oscillator_ECS-2520MV-XXX
