File: board/ice40-dip40.kicad_pcb (KiCad board)
At the start: 4 copper layers, 17.8 x 50.8 mm, 47 parts, among them J1 Conn_02x04_Odd_Even, J2 Conn_01x20, J3 Conn_01x20, J4 USB_B_Micro, SW1 SW_Push, SW2 SW_Push, U1 AT25D081-SSHD, U2 MIC5355-S4YMME, U3 ICE5LP4K-SG48, X1 ECS-2520MV-120-BN-TR

Commit message: Update fpga, flash and oscillator
Parts:
- U1: value AT25D081-SSHD -> W25Q80DVSNIG
- U3: value ICE5LP4K-SG48 -> ICE40UP5K-SG48I
- X1: value ECS-2520MV-120-BN-TR -> ECS-2520MV-160-BN-TR
Changed lines of the file:
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@@
-(kicad_pcb (version 20171130) (host pcbnew 6.0.0-rc1-unknown-r13783-618182dc)
+(kicad_pcb (version 20171130) (host pcbnew 6.0.0-rc1-unknown-r14695-5c055f3f)
   (general
     (thickness 1.6)
@@
       (effects (font (size 1 1) (thickness 0.15)) (justify mirror))
     )
-    (fp_text value AT25D081-SSHD (at 0 -3.5) (layer B.Fab)
+    (fp_text value W25Q80DVSNIG (at 0 -3.5) (layer B.Fab)
       (effects (font (size 1 1) (thickness 0.15)) (justify mirror))
     )
@@
       (effects (font (size 0.8 0.8) (thickness 0.15)))
     )
-    (fp_text value ICE5LP4K-SG48 (at -0.808223 0.987828) (layer F.Fab)
+    (fp_text value ICE40UP5K-SG48I (at -0.808223 0.987828) (layer F.Fab)
       (effects (font (size 0.5 0.5) (thickness 0.125)))
     )
@@
       (effects (font (size 0.8 0.8) (thickness 0.15)) (justify mirror))
     )
-    (fp_text value ECS-2520MV-120-BN-TR (at 0 -1.436841 315) (layer B.Fab)
+    (fp_text value ECS-2520MV-160-BN-TR (at 0 -1.436841 315) (layer B.Fab)
       (effects (font (size 0.5 0.5) (thickness 0.125)) (justify mirror))
     )
